Commit message: robot dog model final + transmission for moving the head

File: experimental_ws/src/exp_assignment2/urdf/robot.xacro (robot description, xacro)
@@ -1,167 +1,180 @@
 <?xml version="1.0"?>
 <robot xmlns:xacro="http://www.ros.org/wiki/xacro" name="robot_xacro">
-<xacro:include filename="$(find exp_assignment2)/urdf/robot.gazebo"/>
-	<xacro:property name="length_wheel" value="0.04" />
-	<xacro:property name="radius_wheel" value="0.1" />
-	<xacro:macro name="default_inertial" params="mass">
-               <inertial>
-                       <mass value="${mass}" />
-                       <origin rpy="0 1.5707 1.5707" xyz="0 0 0"/>
-                       <inertia ixx="0.000526666666667" ixy="0" ixz="0" iyy="0.000526666666667" iyz="0" izz="0.001"/>
-               </inertial>
-	</xacro:macro>
-    <xacro:macro name="wheel_geometry">
-		<geometry>
-       			<cylinder length="${length_wheel}" radius="${radius_wheel}"/>
-     	</geometry>
-	</xacro:macro>
-  <material name="black">
-    <color rgba="0.0 0.0 0.0 1.0"/>
-  </material>
-  <material name="blue">
-    <color rgba="0.203125 0.23828125 0.28515625 1.0"/>
-  </material>
-  <material name="green">
-    <color rgba="0.0 0.8 0.0 1.0"/>
-  </material>
-  <material name="grey">
-    <color rgba="0.2 0.2 0.2 1.0"/>
-  </material>
-  <material name="orange">
-    <color rgba="1.0 0.423529411765 0.0392156862745 1.0"/>
-  </material>
-  <material name="brown">
-    <color rgba="0.870588235294 0.811764705882 0.764705882353 1.0"/>
-  </material>
-  <material name="red">
-    <color rgba="0.80078125 0.12890625 0.1328125 1.0"/>
-  </material>
-  <material name="white">
-    <color rgba="1.0 1.0 1.0 1.0"/>
-  </material>
-	  <link name="link_chassis">
+  <xacro:include filename="$(find exp_assignment2)/urdf/robot.gazebo" />
+  <xacro:property name="length_wheel" value="0.04" />
+  <xacro:property name="radius_wheel" value="0.1" />
+  <xacro:property name="neck_length" value="0.05" />
+  <xacro:property name="neck_radius" value="0.03" />
+  <xacro:macro name="default_inertial" params="mass">
+    <inertial>
+      <mass value="${mass}" />
+      <origin rpy="0 1.5707 1.5707" xyz="0 0 0" />
+      <inertia ixx="0.000526666666667" ixy="0" ixz="0" iyy="0.000526666666667" iyz="0" izz="0.001" />
+    </inertial>
+  </xacro:macro>
+  <xacro:macro name="wheel_geometry">
+    <geometry>
+      <cylinder length="${length_wheel}" radius="${radius_wheel}" />
+    </geometry>
+  </xacro:macro>
+  <link name="link_chassis">
     <!-- pose and inertial -->
     <pose>0 0 0.1 0 0 0</pose>
     <inertial>
-      <mass value="5"/>
-      <origin rpy="0 0 0" xyz="0 0 0.1"/>
-      <inertia ixx="0.0395416666667" ixy="0" ixz="0" iyy="0.106208333333" iyz="0" izz="0.106208333333"/>
+      <mass value="5" />
+      <origin rpy="0 0 0" xyz="0 0 0.1" />
+      <inertia ixx="0.0395416666667" ixy="0" ixz="0" iyy="0.106208333333" iyz="0" izz="0.106208333333" />
     </inertial>
     <!-- body -->
     <collision name="collision_chassis">
       <geometry>
-        <box size="0.5 0.3 0.07"/>
+        <box size="0.5 0.3 0.07" />
       </geometry>
     </collision>
     <visual>
-      <origin rpy="0 0 0" xyz="0 0 0"/>
+      <origin rpy="0 0 0" xyz="0 0 0" />
       <geometry>
-        <box size="0.5 0.3 0.07"/>
+        <box size="0.5 0.3 0.07" />
       </geometry>
-      <material name="blue"/>
+      <material name="blue" />
     </visual>
     <!-- caster front -->
     <collision name="caster_front_collision">
-      <origin rpy=" 0 0 0" xyz="0.35 0 -0.05"/>
+      <origin rpy=" 0 0 0" xyz="0.35 0 -0.05" />
       <geometry>
-        <sphere radius="0.05"/>
+        <sphere radius="0.05" />
       </geometry>
     </collision>
     <visual name="caster_front_visual">
-      <origin rpy=" 0 0 0" xyz="0.2 0 -0.05"/>
+      <origin rpy=" 0 0 0" xyz="0.2 0 -0.05" />
       <geometry>
-        <sphere radius="0.05"/>
+        <sphere radius="0.05" />
       </geometry>
     </visual>
   </link>
-   <link name="link_right_wheel">
-    <xacro:default_inertial mass="0.2"/>
+  <link name="link_right_wheel">
+    <xacro:default_inertial mass="0.2" />
     <collision name="link_right_wheel_collision">
-      <origin rpy="0 1.5707 1.5707" xyz="0 0 0"/>
+      <origin rpy="0 1.5707 1.5707" xyz="0 0 0" />
       <xacro:wheel_geometry />
     </collision>
     <visual name="link_right_wheel_visual">
-      <origin rpy="0 1.5707 1.5707" xyz="0 0 0"/>
+      <origin rpy="0 1.5707 1.5707" xyz="0 0 0" />
       <xacro:wheel_geometry />
-      <material name="red"/>
+      <material name="red" />
     </visual>
   </link>
-   <link name="link_left_wheel">
-    <xacro:default_inertial mass="0.2"/>
+  <link name="link_left_wheel">
+    <xacro:default_inertial mass="0.2" />
     <collision name="link_left_wheel_collision">
-      <origin rpy="0 1.5707 1.5707" xyz="0 0 0"/>
+      <origin rpy="0 1.5707 1.5707" xyz="0 0 0" />
       <xacro:wheel_geometry />
     </collision>
     <visual name="link_left_wheel_visual">
-      <origin rpy="0 1.5707 1.5707" xyz="0 0 0"/>
+      <origin rpy="0 1.5707 1.5707" xyz="0 0 0" />
       <xacro:wheel_geometry />
-      <material name="red"/>
+      <material name="red" />
     </visual>
   </link>
   <joint name="joint_right_wheel" type="continuous">
-    <origin rpy="0 0 0" xyz="-0.05 0.15 0"/>
-    <child link="link_right_wheel"/>
-    <parent link="link_chassis"/>
-    <axis rpy="0 0 0" xyz="0 1 0"/>
-    <limit effort="10000" velocity="1000"/>
-    <joint_properties damping="1.0" friction="1.0"/>
+    <origin rpy="0 0 0" xyz="-0.05 0.15 0" />
+    <child link="link_right_wheel" />
+    <parent link="link_chassis" />
+    <axis rpy="0 0 0" xyz="0 1 0" />
+    <limit effort="10000" velocity="1000" />
+    <joint_properties damping="1.0" friction="1.0" />
   </joint>
   <joint name="joint_left_wheel" type="continuous">
-    <origin rpy="0 0 0" xyz="-0.05 -0.15 0"/>
-    <child link="link_left_wheel"/>
-    <parent link="link_chassis"/>
-    <axis rpy="0 0 0" xyz="0 1 0"/>
-    <limit effort="10000" velocity="1000"/>
-    <joint_properties damping="1.0" friction="1.0"/>
+    <origin rpy="0 0 0" xyz="-0.05 -0.15 0" />
+    <child link="link_left_wheel" />
+    <parent link="link_chassis" />
+    <axis rpy="0 0 0" xyz="0 1 0" />
+    <limit effort="10000" velocity="1000" />
+    <joint_properties damping="1.0" friction="1.0" />
   </joint>
- <link name="neck_link">
-     <xacro:default_inertial mass="0.2"/>
-   <visual>
-     <origin xyz="0 0 0.05" rpy="0 0 0" />
-     <geometry>
-       <cylinder length="0.1" radius="0.02"/>
-     </geometry>
-	<material name="red"/>
-   </visual>
-   <collision>
-     <origin xyz="0 0 0.05" rpy="0 0 0"/>
-     <geometry>
-       <cylinder length="0.1" radius="0.02"/>
-     </geometry>
-   </collision>
- </link>
-   <joint name="neck_joint" type="fixed">
-	    <axis xyz="0 1 0" />
-	    <origin xyz="0.4 0.0 0.15" rpy="0 0 0"/>
-	    <parent link="link_chassis"/>
-	    <child link="neck_link"/>
-	 </joint>
+  <link name="neck_link">
+    <xacro:default_inertial mass="0.05" />
+    <visual>
+      <origin xyz="0 0 ${neck_length/2}" rpy="0 0 0" />
+      <geometry>
+        <cylinder length="${neck_length}" radius="${neck_radius}" />
+      </geometry>
+      <material name="red" />
+    </visual>
+    <collision>
+      <origin xyz="0 0 ${neck_length/2}" rpy="0 0 0" />
+      <geometry>
+        <cylinder length="${neck_length}" radius="${neck_radius}" />
+      </geometry>
+    </collision>
+  </link>
+  <joint name="neck_joint" type="fixed">
+    <axis xyz="0 1 0" />
+    <origin xyz="0.2 0.0 0.015" rpy="0 0 0" />
+    <parent link="link_chassis" />
+    <child link="neck_link" />
+  </joint>
+  <!-- head definition -->
+  <link name="head_link">
+    <xacro:default_inertial mass="0.2" />
+    <collision>
+      <origin xyz="0 0 0.06" rpy="0 0 0" /> <!-- frame moved to the base of the head -->
+      <geometry>
+        <box size="0.2 0.12 0.12" />
+      </geometry>
+    </collision>
+    <visual>
+      <origin xyz="0 0 0.06" rpy="0 0 0" /> <!-- frame moved to the base of the head -->
+      <geometry>
+        <box size="0.2 0.12 0.12" />
+      </geometry>
+      <material name="red" />
+    </visual>
+  </link>
+  <joint name="head_joint" type="revolute">
+    <axis xyz="0 0 1" />
+    <limit effort="1000.0" lower="-1.8" upper="1.8" velocity="0.5" />
+    <origin rpy="0 0 0" xyz="0.03 0 ${neck_length}" />
+    <parent link="neck_link" />
+    <child link="head_link" />
+  </joint>
+  <!-- transmission -->
+  <transmission name="head_joint_trans">
+    <type>transmission_interface/SimpleTransmission</type>
+    <joint name="head_joint">
+      <hardwareInterface>hardware_interface/EffortJointInterface</hardwareInterface>
+    </joint>
+    <actuator name="motor1">
+      <hardwareInterface>hardware_interface/EffortJointInterface</hardwareInterface>
+      <mechanicalInterface>1</mechanicalInterface>
+    </actuator>
+  </transmission>
   <link name="camera_link">
-	    <collision>
-	      <origin xyz="0 0 0.25" rpy="0 0 0"/>
-	      <geometry>
-		<box size="0.05 0.05 0.05"/>
-	      </geometry>
-	    </collision>
-	    <visual>
-	      <origin xyz="0 0 0.25" rpy="0 0 0"/>
-	      <geometry>
-		<box size="0.05 0.05 0.05"/>
-	      </geometry>
-	      <material name="red">
-		<color rgba="1 0 0 1"/>
-	      </material>
-	    </visual>
-	    <inertial>
-	      <mass value="1e-5" />
-	      <origin xyz="0 0 0" rpy="0 0 0"/>
-	      <inertia ixx="1e-6" ixy="0" ixz="0" iyy="1e-6" iyz="0" izz="1e-6" />
-	    </inertial>
+    <collision>
+      <origin xyz="0 0 0" rpy="0 0 0" />
+      <geometry>
+        <box size="0.05 0.05 0.05" />
+      </geometry>
+    </collision>
+    <visual>
+      <origin xyz="0 0 0" rpy="0 0 0" />
+      <geometry>
+        <box size="0.05 0.05 0.05" />
+      </geometry>
+      <material name="red">
+        <color rgba="1 0 0 1" />
+      </material>
+    </visual>
+    <inertial>
+      <mass value="1e-5" />
+      <origin xyz="0 0 0" rpy="0 0 0" />
+      <inertia ixx="1e-6" ixy="0" ixz="0" iyy="1e-6" iyz="0" izz="1e-6" />
+    </inertial>
   </link>
   <joint name="camera_joint" type="fixed">
-	    <axis xyz="0 1 0" />
-	    <origin xyz="0 0 0.1" rpy="0 0 0"/>
-	    <parent link="neck_link"/>
-	    <child link="camera_link"/>
-	 </joint>
+    <axis xyz="0 1 0" />
+    <origin xyz="0.075 0 0.145" rpy="0 0 0" />
+    <parent link="head_link" />
+    <child link="camera_link" />
+  </joint>
 </robot>
